File: res/one_of_each.kicad_sch (KiCad schematic)
At the start: 3 parts

Commit message: Convert grid to schematic with footprints.
Parts:
- R?: footprint (none) -> Resistor_SMD:R_01005_0402Metric
- T? (x2): footprint (none) -> Package_TO_SOT_SMD:SOT-23
Changed lines of the file:
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@@
       (effects (font (size 1.27 1.27)))
     )
-    (property "Footprint" "" (at 59.69 44.45 0)
+    (property "Footprint" "Package_TO_SOT_SMD:SOT-23" (at 59.69 44.45 0)
       (effects (font (size 1.27 1.27)) hide)
     )
@@
       (effects (font (size 1.27 1.27)))
     )
-    (property "Footprint" "" (at 52.07 44.45 0)
+    (property "Footprint" "Package_TO_SOT_SMD:SOT-23" (at 52.07 44.45 0)
       (effects (font (size 1.27 1.27)) hide)
     )
@@
       (effects (font (size 1.27 1.27)) (justify left))
     )
-    (property "Footprint" "" (at 35.56 44.45 0)
+    (property "Footprint" "Resistor_SMD:R_01005_0402Metric" (at 35.56 44.45 0)
       (effects (font (size 1.27 1.27)) hide)
     )
